Commit message: add wall to rviz

File: src/robot_arm/urdf/arm.urdf (robot description, URDF)
Before this commit: robot arm, 7 links, 6 joints
Joints:
- joint world_joint: origin xyz=0.0 0.0 0.0 rpy=0.0 0.0 0.0 -> xyz=2.5 6.0 4.0 rpy=3.1416 0.0 0.0

Commit message: Add arm URDF

File: src/robot_arm/urdf/arm.urdf (robot description, URDF)
Before this commit: robot arm, 7 links, 6 joints
Links:
- removed link forearm_link
- removed link shoulder_link
- removed link upper_arm_link
- removed link wrist_1_link
- added link elbow_link, mass 1.219; collision sphere radius=0.12; visual sphere radius=0.12
- added link main_arm_link, mass 2.275; collision box size=0.1 0.1 7; visual box size=0.1 0.1 7
- added link secondary_arm_link, mass 1.219; collision box size=3.2 0.07 0.07; visual box size=3.2 0.07 0.07
- added link shoulder_link_1; collision cylinder length=0.1 radius=0.4; visual cylinder length=0.1 radius=0.4
- added link shoulder_link_2, mass 8.393; collision cylinder length=0.1 radius=0.4; visual cylinder length=0.1 radius=0.4
- added link third_arm_link, mass 1.219; collision box size=0.2 0.05 0.05; visual box size=0.2 0.05 0.05
- link base_link: mass 4.0 -> None; geometry 
- link ee_link: mass None -> 1.219; geometry collision sphere radius=0.08; visual sphere radius=0.08
Joints:
- removed joint ee_fixed_joint
- removed joint elbow_joint
- removed joint shoulder_lift_joint
- removed joint shoulder_pan_joint
- removed joint world_joint
- removed joint wrist_1_joint
- added joint base_join: type fixed, parent world, child base_link, origin xyz=2.5 6.0 4.0 rpy=3.14159265 0.0 0.0
- added joint ee_join: type fixed, parent third_arm_link, child ee_link, origin xyz=0.2 0.0 0.0 rpy=0.0 0.0 0
- added joint elbow_join_1: type revolute, parent main_arm_link, child elbow_link, origin xyz=0.0 0.0 0.0 rpy=-1.570796325 0.0 0.0, axis 0 0 1, limit lower=-3.14159265 upper=3.14159265 effort=28.0 velocity=3.2
- added joint elbow_join_2: type revolute, parent elbow_link, child secondary_arm_link, origin xyz=0.0 0.0 0.0 rpy=0.0 -1.570796325 0.0, axis 0 0 1, limit lower=-1.570796325 upper=1.570796325 effort=28.0 velocity=3.2
- added joint main_arm_join: type prismatic, parent shoulder_link_2, child main_arm_link, origin xyz=0.5 0.0 0.0 rpy=0.0 1.570796325 0.0, axis 0 0 1, limit lower=0.0 upper=6.5 effort=150.0 velocity=2
- added joint second_last_join: type fixed, parent secondary_arm_link, child third_arm_link, origin xyz=3.0 0.0 0.0 rpy=0.0 0.0 -1.570796325
- added joint shoulder_join_1: type revolute, parent base_link, child shoulder_link_1, origin xyz=0.0 0.0 0.0 rpy=0.0 0.0 0.0, axis 0 0 1, limit lower=-3.14159265 upper=3.14159265 effort=150.0 velocity=3.15
- added joint shoulder_join_2: type revolute, parent shoulder_link_1, child shoulder_link_2, origin xyz=0.0 0.0 0.0 rpy=1.570796325 0.0 0.0, axis 0 0 1, limit lower=0.0 upper=3.14159265 effort=150.0 velocity=3.15

Commit message: Add dynamics

File: src/robot_arm/urdf/arm.urdf (robot description, URDF)
Before this commit: robot arm, 9 links, 8 joints
Links:
- link base_link: mass None -> 10.0
- link shoulder_link_1: mass None -> 8.393
Joints:
- joint main_arm_join: limit lower=0.0 upper=6.5 effort=150.0 velocity=2 -> lower=0.0 upper=6.5 effort=1500000000.0 velocity=2

Commit message: update urdf model

File: src/robot_arm/urdf/arm.urdf (robot description, URDF)
Before this commit: robot arm, 9 links, 8 joints
Links:
- link base_link: mass 10.0 -> None
Joints:
- joint elbow_join_1: limit lower=-3.14159265 upper=3.14159265 effort=28.0 velocity=3.2 -> effort=28.0 velocity=3.2
- joint elbow_join_2: limit lower=-1.570796325 upper=1.570796325 effort=28.0 velocity=3.2 -> effort=28.0 velocity=3.2
- joint main_arm_join: limit lower=0.0 upper=6.5 effort=1500000000.0 velocity=2 -> lower=0.0 upper=1 effort=15000000000000.0 velocity=2

Commit message: Add stopping

File: src/robot_arm/urdf/arm.urdf (robot description, URDF)
Before this commit: robot arm, 9 links, 8 joints
Joints:
- joint elbow_join_1: limit effort=28.0 velocity=3.2 -> lower=-3.14159265 upper=3.14159265 effort=28.0 velocity=3.2
- joint elbow_join_2: limit effort=28.0 velocity=3.2 -> lower=-1.570796325 upper=1.570796325 effort=28.0 velocity=3.2
- joint main_arm_join: limit lower=0.0 upper=1 effort=15000000000000.0 velocity=2 -> lower=0.0 upper=1 effort=150.0 velocity=2

Commit message: finish part 3

File: src/robot_arm/urdf/arm.urdf (robot description, URDF)
Before this commit: robot arm, 9 links, 8 joints
Links:
- link ee_link: mass 1.219 -> 0.2
- link elbow_link: mass 1.219 -> 1.0
- link main_arm_link: mass 2.275 -> 5
- link secondary_arm_link: mass 1.219 -> 1.0
- link shoulder_link_1: mass 8.393 -> 3.0
- link shoulder_link_2: mass 8.393 -> 3.0
- link third_arm_link: mass 1.219 -> 0.2
Joints:
- joint elbow_join_1: limit lower=-3.14159265 upper=3.14159265 effort=28.0 velocity=3.2 -> lower=-3.14159265 upper=3.14159265 effort=100.0 velocity=3.2
- joint elbow_join_2: limit lower=-1.570796325 upper=1.570796325 effort=28.0 velocity=3.2 -> lower=-1.570796325 upper=1.570796325 effort=100.0 velocity=3.2
- joint main_arm_join: limit lower=0.0 upper=1 effort=150.0 velocity=2 -> lower=0.0 upper=6 effort=10000.0 velocity=2
- joint shoulder_join_1: limit lower=-3.14159265 upper=3.14159265 effort=150.0 velocity=3.15 -> lower=-3.14159265 upper=3.14159265 effort=10000.0 velocity=3.15
- joint shoulder_join_2: limit lower=0.0 upper=3.14159265 effort=150.0 velocity=3.15 -> lower=-0.523599 upper=3.66519 effort=10000.0 velocity=3.15

Commit message: Finish robot

File: src/robot_arm/urdf/arm.urdf (robot description, URDF)
Before this commit: robot arm, 9 links, 8 joints
Links:
- link secondary_arm_link: geometry collision box size=3.2 0.07 0.07; visual box size=2.2 0.07 0.07
Joints:
- joint second_last_join: origin xyz=3.0 0.0 0.0 rpy=0.0 0.0 -1.570796325 -> xyz=2.0 0.0 0.0 rpy=0.0 0.0 -1.570796325
